Commit message: feat: divide vision tesground into several .xacro files

File: ros/src/gazebo_worlds/worlds/vision_testground/aux_macros.xacro (robot description, xacro)
@@ -62,4 +62,5 @@
     <model name="cylinder">
     <!-- Raised by half the height so the base rests on the ground plane -->
+        <static>true</static>
         <pose>${x} ${y} ${cylinder_height / 2} 0 0 0</pose>
         <link name="cylinder_${name}">

File: ros/src/gazebo_worlds/worlds/vision_testground/common_properties.xacro (robot description, xacro)
@@ -34,9 +34,9 @@
   <xacro:property name="EAST"  value="3"/>
   <xacro:property name="SOUTH" value="2"/>
-  <xacro:property name="cylinder_height" value="0.08"/>
-  <xacro:property name="cylinder_radius" value="0.08"/>
+  <xacro:property name="box_size"     value="0.02"/>
+  <xacro:property name="box_mass"     value="0.02"/>
+  <xacro:property name="cylinder_height" value="0.1"/>
+  <xacro:property name="cylinder_radius" value="${box_size}"/>
   <xacro:property name="arrow_base_z" value="0.5"/>
-  <xacro:property name="box_size"     value="0.08"/>
-  <xacro:property name="box_mass"     value="0.02"/>
   <xacro:property name="spacing"      value="0.4"/>
 </sdf>

Commit message: fix: Cylinder name

File: ros/src/gazebo_worlds/worlds/vision_testground/aux_macros.xacro (robot description, xacro)
@@ -60,9 +60,9 @@
   <!-- Small cube resting on the floor. Inertia is computed from the mass and size. -->
   <xacro:macro name="box" params="name x y rgb">
-    <model name="cylinder">
+    <model name="cylinder_${name}">
     <!-- Raised by half the height so the base rests on the ground plane -->
         <static>true</static>
         <pose>${x} ${y} ${cylinder_height / 2} 0 0 0</pose>
-        <link name="cylinder_${name}">
+        <link name="cylinder">
             <collision name="cylinder_collision">
                 <geometry>

File: ros/src/gazebo_worlds/worlds/vision_testground/vision_testground.world.xacro (robot description, xacro)
@@ -58,5 +58,7 @@
         <xacro:entry_outer x="-9" y="0" px="${SOUTH}" />
         <!-- OUTER WALL END -->
-        <xacro:box x="${9*0.32}" y="0" name ="1" rgb="1 0 0"/>
+        <xacro:box x="${7*0.32}" y="${1*0.32}"  name ="r1" rgb="1 0 0"/>
+        <xacro:box x="${7*0.32}" y="${0*0.32}"  name ="b1" rgb="0 0 1"/>
+        <xacro:box x="${7*0.32}" y="${-1*0.32}" name ="g1" rgb="0 1 0"/>
         <!--xacro:arrow x="1" y="-1" px="0" pd="1" L="0.030" r="1" g="0" b="0" /-->
         <!--xacro:arrow x="1" y="0"  px="0" pd="1" L="0.060" r="0" g="1" b="0" /-->
